Commit message: Add mesh geometry

File: data/minis.urdf (robot description, URDF)
Before this commit: robot quadruped, 55 links, 54 joints
Links:
- link aiy0_center_link: geometry visual mesh filename=meshes/SR319-AIY.stl scale=1 1 1
- link arm0_left_link: geometry visual mesh filename=meshes/SR319-SERVO.stl scale=1 1 1
- link arm0_right_link: geometry visual mesh filename=meshes/SR319-SERVO.stl scale=1 1 1
- link arm1_left_link: geometry visual mesh filename=meshes/SR319-SERVO-ROTOR.stl scale=1 1 1
- link arm1_right_link: geometry visual mesh filename=meshes/SR319-SERVO-ROTOR.stl scale=1 1 1
- link arm2_left_link: geometry visual mesh filename=meshes/SR319-20x55-ASSEMBLY.stl scale=1 1 1
- link arm2_right_link: geometry visual mesh filename=meshes/SR319-20x55-ASSEMBLY.stl scale=1 1 1
- link arm3_left_link: geometry visual mesh filename=meshes/SR319-SERVO.stl scale=1 1 1
- link arm3_right_link: geometry visual mesh filename=meshes/SR319-SERVO.stl scale=1 1 1
- link arm4_left_link: geometry visual mesh filename=meshes/SR319-20x43.stl scale=1 1 1
- link arm4_right_link: geometry visual mesh filename=meshes/SR319-20x43.stl scale=1 1 1
- link arm5_left_link: geometry visual mesh filename=meshes/SR319-20x43.stl scale=1 1 1
- link arm5_right_link: geometry visual mesh filename=meshes/SR319-20x43.stl scale=1 1 1
- link arm6_left_link: geometry visual mesh filename=meshes/SR319-SERVO.stl scale=1 1 1
- link arm6_right_link: geometry visual mesh filename=meshes/SR319-SERVO.stl scale=1 1 1
- link arm7_left_link: geometry visual mesh filename=meshes/SR319-20x55-ASSEMBLY.stl scale=1 1 1
- link arm7_right_link: geometry visual mesh filename=meshes/SR319-20x55-ASSEMBLY.stl scale=1 1 1
- link arm8_left_link: geometry collision box size=0.040165 0.020165 0.001500; visual mesh filename=meshes/SR319-HOE.stl scale=1 1 1
- link arm8_right_link: geometry collision box size=0.040165 0.020165 0.001500; visual mesh filename=meshes/SR319-HOE.stl scale=1 1 1
- link battery_link: geometry visual mesh filename=meshes/SR319-BATTERY.stl scale=1 1 1
- link cam0_center_link: geometry visual mesh filename=meshes/SR319-CAM.stl scale=1 1 1
- link cam0_left_link: geometry visual mesh filename=meshes/SR319-CAM.stl scale=1 1 1
- link cam0_right_link: geometry visual mesh filename=meshes/SR319-CAM.stl scale=1 1 1
- link chassis_center_link: geometry visual mesh filename=meshes/SR319-BODY.stl scale=1 1 1
- link head0_center_link: geometry visual mesh filename=meshes/SR319-20x43.stl scale=1 1 1
- link head1_center_link: geometry visual mesh filename=meshes/SR319-SERVO-ROTOR.stl scale=1 1 1
- link head2_center_link: geometry visual mesh filename=meshes/SR319-SERVO.stl scale=1 1 1
- link leg0_left_link: geometry visual mesh filename=meshes/SR319-SERVO.stl scale=1 1 1
- link leg0_right_link: geometry visual mesh filename=meshes/SR319-SERVO.stl scale=1 1 1
- link leg10_left_link: geometry visual mesh filename=meshes/SR319-20x55-ASSEMBLY.stl scale=1 1 1
- link leg10_right_link: geometry visual mesh filename=meshes/SR319-20x55-ASSEMBLY.stl scale=1 1 1
- link leg11_left_link: geometry visual mesh filename=meshes/SR319-20x55-ASSEMBLY.stl scale=1 1 1
- link leg11_right_link: geometry visual mesh filename=meshes/SR319-20x55-ASSEMBLY.stl scale=1 1 1
- link leg12_left_link: geometry visual mesh filename=meshes/SR319-SERVO.stl scale=1 1 1
- link leg12_right_link: geometry visual mesh filename=meshes/SR319-SERVO.stl scale=1 1 1
- link leg13_left_link: geometry collision box size=0.001534 0.048000 0.015582; visual mesh filename=meshes/SR319-FEET.stl scale=1 1 1
- link leg13_right_link: geometry collision box size=0.001534 0.048000 0.015582; visual mesh filename=meshes/SR319-FEET.stl scale=1 1 1
- link leg1_left_link: geometry visual mesh filename=meshes/SR319-20x55-ASSEMBLY.stl scale=1 1 1
- link leg1_right_link: geometry visual mesh filename=meshes/SR319-20x55-ASSEMBLY.stl scale=1 1 1
- link leg2_left_link: geometry visual mesh filename=meshes/SR319-40x43.stl scale=1 1 1
- link leg2_right_link: geometry visual mesh filename=meshes/SR319-40x43.stl scale=1 1 1
- link leg3_left_link: geometry visual mesh filename=meshes/SR319-SERVO.stl scale=1 1 1
- link leg3_right_link: geometry visual mesh filename=meshes/SR319-SERVO.stl scale=1 1 1
- link leg4_left_link: geometry visual mesh filename=meshes/SR319-20x55-ASSEMBLY.stl scale=1 1 1
- link leg4_right_link: geometry visual mesh filename=meshes/SR319-20x55-ASSEMBLY.stl scale=1 1 1
- link leg5_left_link: geometry visual mesh filename=meshes/SR319-20x43.stl scale=1 1 1
- link leg5_right_link: geometry visual mesh filename=meshes/SR319-20x43.stl scale=1 1 1
- link leg6_left_link: geometry visual mesh filename=meshes/SR319-SERVO.stl scale=1 1 1
- link leg6_right_link: geometry visual mesh filename=meshes/SR319-SERVO.stl scale=1 1 1
- link leg7_left_link: geometry visual mesh filename=meshes/SR319-20x55-ASSEMBLY.stl scale=1 1 1
- link leg7_right_link: geometry visual mesh filename=meshes/SR319-20x55-ASSEMBLY.stl scale=1 1 1
- link leg8_left_link: geometry visual mesh filename=meshes/SR319-20x43.stl scale=1 1 1
- link leg8_right_link: geometry visual mesh filename=meshes/SR319-20x43.stl scale=1 1 1
- link leg9_left_link: geometry visual mesh filename=meshes/SR319-SERVO.stl scale=1 1 1
- link leg9_right_link: geometry visual mesh filename=meshes/SR319-SERVO.stl scale=1 1 1

Commit message: Add .obj meshes, change collision to body from battery

File: data/minis.urdf (robot description, URDF)
Before this commit: robot quadruped, 55 links, 54 joints
Links:
- link chassis_center_link: geometry collision box size=0.001500 0.121124 0.140800; visual mesh filename=meshes/SR319-BODY.stl scale=1 1 1

Commit message: Makes collisions thicker, fixes shapes

File: data/minis.urdf (robot description, URDF)
Before this commit: robot quadruped, 55 links, 54 joints
Links:
- link aiy0_center_link: geometry visual box size=0.080330 0.087165 0.046330
- link arm0_left_link: geometry visual box size=0.020132 0.040332 0.048600
- link arm0_right_link: geometry visual box size=0.020132 0.040332 0.048600
- link arm1_left_link: geometry 
- link arm1_right_link: geometry 
- link arm2_left_link: geometry 
- link arm2_right_link: geometry 
- link arm3_left_link: geometry visual box size=0.020132 0.040332 0.048600
- link arm3_right_link: geometry visual box size=0.020132 0.040332 0.048600
- link arm4_left_link: geometry 
- link arm4_right_link: geometry 
- link arm5_left_link: geometry 
- link arm5_right_link: geometry 
- link arm6_left_link: geometry visual box size=0.020132 0.040332 0.048600
- link arm6_right_link: geometry visual box size=0.020132 0.040332 0.048600
- link arm7_left_link: geometry 
- link arm7_right_link: geometry 
- link arm8_left_link: geometry collision box size=0.040165 0.021665 0.060479; visual box size=0.040165 0.021665 0.060479
- link arm8_right_link: geometry collision box size=0.040165 0.021665 0.060479; visual box size=0.040165 0.021665 0.060479
- link battery_link: geometry 
- link cam0_center_link: geometry visual box size=0.040659 0.031214 0.030049
- link cam0_left_link: geometry visual box size=0.040659 0.031214 0.030049
- link cam0_right_link: geometry visual box size=0.040659 0.031214 0.030049
- link chassis_center_link: geometry collision box size=0.045353 0.121569 0.143882; visual box size=0.045353 0.121569 0.143882
- link head0_center_link: geometry 
- link head1_center_link: geometry 
- link head2_center_link: geometry visual box size=0.020132 0.040332 0.048600
- link leg0_left_link: geometry visual box size=0.020132 0.040332 0.048600
- link leg0_right_link: geometry visual box size=0.020132 0.040332 0.048600
- link leg10_left_link: geometry 
- link leg10_right_link: geometry 
- link leg11_left_link: geometry 
- link leg11_right_link: geometry 
- link leg12_left_link: geometry visual box size=0.020132 0.040332 0.048600
- link leg12_right_link: geometry visual box size=0.020132 0.040332 0.048600
- link leg13_left_link: geometry collision box size=0.119989 0.074470 0.017165; visual box size=0.119989 0.074470 0.017165
- link leg13_right_link: geometry collision box size=0.119989 0.074470 0.017165; visual box size=0.119989 0.074470 0.017165
- link leg1_left_link: geometry 
- link leg1_right_link: geometry 
- link leg2_left_link: geometry 
- link leg2_right_link: geometry 
- link leg3_left_link: geometry visual box size=0.020132 0.040332 0.048600
- link leg3_right_link: geometry visual box size=0.020132 0.040332 0.048600
- link leg4_left_link: geometry 
- link leg4_right_link: geometry 
- link leg5_left_link: geometry 
- link leg5_right_link: geometry 
- link leg6_left_link: geometry visual box size=0.020132 0.040332 0.048600
- link leg6_right_link: geometry visual box size=0.020132 0.040332 0.048600
- link leg7_left_link: geometry 
- link leg7_right_link: geometry 
- link leg8_left_link: geometry 
- link leg8_right_link: geometry 
- link leg9_left_link: geometry visual box size=0.020132 0.040332 0.048600
- link leg9_right_link: geometry visual box size=0.020132 0.040332 0.048600

Commit message: Adds merge_fixed_links model optimizer

File: data/minis.urdf (robot description, URDF)
Before this commit: robot quadruped, 55 links, 54 joints
Links:
- removed link arm0_left_link
- removed link arm0_right_link
- removed link arm2_left_link
- removed link arm2_right_link
- removed link arm4_left_link
- removed link arm4_right_link
- removed link arm5_left_link
- removed link arm5_right_link
- removed link arm6_left_link
- removed link arm6_right_link
- removed link battery_link
- removed link cam0_center_link
- removed link cam0_left_link
- removed link cam0_right_link
- removed link head0_center_link
- removed link head1_center_link
- removed link leg0_left_link
- removed link leg0_right_link
- removed link leg11_left_link
- removed link leg11_right_link
- removed link leg2_left_link
- removed link leg2_right_link
- removed link leg3_left_link
- removed link leg3_right_link
- removed link leg5_left_link
- removed link leg5_right_link
- removed link leg6_left_link
- removed link leg6_right_link
- removed link leg8_left_link
- removed link leg8_right_link
- removed link leg9_left_link
- removed link leg9_right_link
- link aiy0_center_link: geometry collision box size=0.080330 0.087165 0.046330; visual box size=0.080330 0.087165 0.046330
Joints:
- removed joint arm0_left_joint
- removed joint arm0_right_joint
- removed joint arm2_left_joint
- removed joint arm2_right_joint
- removed joint arm4_left_joint
- removed joint arm4_right_joint
- removed joint arm5_left_joint
- removed joint arm5_right_joint
- removed joint arm6_left_joint
- removed joint arm6_right_joint
- removed joint battery_joint
- removed joint cam0_center_joint
- removed joint cam0_left_joint
- removed joint cam0_right_joint
- removed joint head0_center_joint
- removed joint head1_center_joint
- removed joint leg0_left_joint
- removed joint leg0_right_joint
- removed joint leg11_left_joint
- removed joint leg11_right_joint
- removed joint leg2_left_joint
- removed joint leg2_right_joint
- removed joint leg3_left_joint
- removed joint leg3_right_joint
- removed joint leg5_left_joint
- removed joint leg5_right_joint
- removed joint leg6_left_joint
- removed joint leg6_right_joint
- removed joint leg8_left_joint
- removed joint leg8_right_joint
- removed joint leg9_left_joint
- removed joint leg9_right_joint
- joint arm1_left_joint: origin xyz=0.0 0.0 0.009 rpy=3.141592 0.0 1.570796 -> xyz=-1.000000e-03 1.020000e-01 7.720000e-02 rpy=3.141592e+00 -0.000000e+00 1.570796e+00; parent arm0_left_link -> chassis_center_link
- joint arm1_right_joint: origin xyz=0.0 0.0 0.009 rpy=3.141592 0.0 1.570796 -> xyz=-9.99994118e-04 1.02000000e-01 -7.72000000e-02 rpy=-1.30717959e-06 2.13589809e-13 1.57079665e+00; parent arm0_right_link -> chassis_center_link
- joint arm3_left_joint: origin xyz=0.0 0.0 0.00 rpy=0.0 0.0 -1.570796 -> xyz=0. -0.0169 -0.022 rpy=0.78539816 1.57079586 -0.78539816; parent arm2_left_link -> arm1_left_link
- joint arm3_right_joint: origin xyz=0.0 0.0 0.00 rpy=0.0 0.0 -1.570796 -> xyz=0. -0.0169 -0.022 rpy=0.78539816 1.57079586 -0.78539816; parent arm2_right_link -> arm1_right_link
- joint arm7_left_joint: origin xyz=0.0 0.00 0.00 rpy=0.0 0.0 0.0 -> xyz=-1.24182117e-08 -7.60000176e-02 -3.71182147e-08 rpy=-1.30358979e-06 -3.26794900e-07 3.14159233e+00; parent arm6_left_link -> arm3_left_link
- joint arm7_right_joint: origin xyz=0.0 0.00 0.00 rpy=0.0 0.0 0.0 -> xyz=-1.24182117e-08 -7.60000176e-02 -3.71182147e-08 rpy=-1.30358979e-06 -3.26794900e-07 3.14159233e+00; parent arm6_right_link -> arm3_right_link
- joint head2_center_joint: origin xyz=0.0 0.0 0.009 rpy=0.0 3.141592 -1.570796 -> xyz=-9.99994118e-04 1.06000000e-01 -2.90884593e-09 rpy=2.36165719e+00 -1.57079586e+00 -7.90861513e-01; parent head1_center_link -> chassis_center_link
- joint leg10_left_joint: origin xyz=0.0 0.00 0.00 rpy=0.0 0.0 0.0 -> xyz=1.24182041e-08 5.99999941e-02 1.00001242e-03 rpy=1.74886971e-20 3.26794897e-07 -3.26794790e-07; parent leg9_left_link -> leg7_left_link
- joint leg10_right_joint: origin xyz=0.0 0.00 0.00 rpy=0.0 0.0 0.0 -> xyz=1.24182041e-08 5.99999941e-02 1.00001242e-03 rpy=1.74886971e-20 3.26794897e-07 -3.26794790e-07; parent leg9_right_link -> leg7_right_link
- joint leg12_left_joint: origin xyz=0.0 0.0 0.00 rpy=0.0 0.0 1.570796 -> xyz=-2.00000000e-02 4.40000000e-02 -2.00000000e-02 rpy=1.57079600e+00 3.26794897e-07 -1.57079698e+00; parent leg11_left_link -> leg10_left_link
- joint leg12_right_joint: origin xyz=0.0 0.0 0.00 rpy=0.0 0.0 1.570796 -> xyz=-2.00000000e-02 4.40000000e-02 -2.00000000e-02 rpy=1.57079600e+00 3.26794897e-07 -1.57079698e+00; parent leg11_right_link -> leg10_right_link
- joint leg1_left_joint: origin xyz=0.0 0.0 0.0 rpy=0.0 0.0 1.570796 -> xyz=0.018 0. 0.033 rpy=0.78539816 -1.57079586 2.35619416; parent leg0_left_link -> chassis_center_link
- joint leg1_right_joint: origin xyz=0.0 0.0 0.0 rpy=0.0 0.0 1.570796 -> xyz=-0.018 0. -0.033 rpy=-0.78539816 1.57079586 2.35619416; parent leg0_right_link -> chassis_center_link
- joint leg4_left_joint: origin xyz=0.0 0.0 0.0 rpy=0.0 0.0 1.570796 -> xyz=1.80000000e-02 3.80000033e-02 -2.69999948e-02 rpy=-3.26794898e-07 1.57079633e+00 0.00000000e+00; parent leg3_left_link -> leg1_left_link
- joint leg4_right_joint: origin xyz=0.0 0.0 0.0 rpy=0.0 0.0 1.570796 -> xyz=-0.01800001 0.038 -0.00700002 rpy=3.14159233 -1.57079567 -3.14159265; parent leg3_right_link -> leg1_right_link
- joint leg7_left_joint: origin xyz=0.0 0.0 0.0 rpy=0.0 0.0 0.0 -> xyz=1.24182080e-08 6.00000059e-02 -3.49999876e-02 rpy=3.14159200e+00 3.26794897e-07 3.14159233e+00; parent leg6_left_link -> leg4_left_link
- joint leg7_right_joint: origin xyz=0.0 0.0 0.0 rpy=0.0 0.0 0.0 -> xyz=1.24182041e-08 5.99999941e-02 1.00001242e-03 rpy=1.74886971e-20 3.26794897e-07 -3.26794790e-07; parent leg6_right_link -> leg4_right_link
